Commit message: map generating...

File: urdf/robot_core.urdf.xacro (robot description, xacro)
@@ -5,5 +5,5 @@
     <xacro:include filename="$(find mobile_robot)/urdf/camera.xacro"/>
     <xacro:include filename="$(find mobile_robot)/urdf/imu_plugin.xacro"/>
-    <xacro:include filename="$(find mobile_robot)/description/gazebo_control.xacro"/>
+    <!-- <xacro:include filename="$(find mobile_robot)/description/gazebo_control.xacro"/> -->
     <gazebo>
         <plugin name="gazebo_ros_control" filename="libgazebo_ros_control.so">

File: urdf/rover.urdf.xacro (robot description, xacro)
@@ -17,5 +17,5 @@
     <link name="base_link">
     </link>
-    <!-- <joint name="base_footprint_joint" type="fixed">
+    <joint name="base_footprint_joint" type="fixed">
         <parent link="base_link"/>
         <child link="base_footprint"/>
@@ -23,5 +23,5 @@
     </joint>
     <link name="base_footprint">
-    </link> -->
+    </link>
     <joint name="Chassis_joint" type="fixed">
         <parent link="base_link"/>
@@ -115,5 +115,5 @@
         <visual>
             <geometry>
-                <mesh filename="${path}" scale="0.005 0.005 0.005"/> #length = 0.0182 radius = "0.0660"
+                <mesh filename="${path}" scale="0.005 0.005 0.005"/> #length = 0.0182 radius = "0.0330"
             </geometry>
             <material name="">
