Commit message: implemented a 4wheel_bot

File: urdf/lidar.xacro (robot description, xacro)
@@ -1,4 +1,4 @@
 <?xml version="1.0"?>
-<robot xmlns:xacro="http://www.ros.org/wiki/xacro">
+<robot xmlns:xacro="http://www.ros.org/wiki/xacro" name="my_rover">
     <!-- camera/sensor mount -->
     <joint name="lidar_joint" type="fixed">
@@ -26,11 +26,8 @@
             <mass value="0.1"/>
             <origin xyz="0.0 0.0 0.0" rpy="0.0 0.0 0.0"/>
-            <inertia ixx="${(1/12) * mass * (3*radius*radius + length*length)}" ixy="0.0" ixz="0.0"
-                    iyy="${(1/12) * mass * (3*radius*radius + length*length)}" iyz="0.0"
-                    izz="${(1/12) * mass * (radius*radius)}" />
+            <inertia ixx="0.00024" ixy="0.0" ixz="0.0"
+                    iyy="0.00024" iyz="0.0"
+                    izz="0.00005" />
         </inertial>
-    </link>
-    <gazebo reference = "lidar_link">
-        <material> Gazebo/Blue </material>
         <sensor name = "laser" type = "ray">
             <pose> 0 0 0 0 0 0 </pose>
@@ -40,5 +37,5 @@
                 <scan>
                     <horizontal>
-                        <samples>720</samples>
+                        <samples>360</samples>
                         <resolution>1</resolution>
                         <min_angle>-2.356194</min_angle>  <!-- -135 degrees in radians -->
@@ -52,5 +49,5 @@
                 </range>
             </ray>
-            <plugin name="laser_controller" filename="libgazebo_ros_ray_sensor.so">
+            <plugin name="laser" filename="libgazebo_ros_ray_sensor.so">
                 <ros>
                     <argument>~/out:=scan</argument>
@@ -60,4 +57,7 @@
             </plugin>
         </sensor>
+    </link>
+    <gazebo reference = "lidar_link">
+        <material> Gazebo/Blue </material>
     </gazebo>
 </robot>

File: urdf/robot_core.xacro (robot description, xacro)
@@ -2,5 +2,5 @@
 <robot xmlns:xacro="http://www.ros.org/wiki/xacro" name="my_rover">
     <xacro:include filename="$(find mobile_robot)/urdf/rover.urdf.xacro"/>
-    <!-- <xacro:include filename="$(find mobile_robot)/description/gazebo_control.xacro"/> -->
     <xacro:include filename="$(find mobile_robot)/urdf/lidar.xacro"/>
+    <xacro:include filename="$(find mobile_robot)/description/transmission.urdf"/>
 </robot>

File: urdf/rover.urdf.xacro (robot description, xacro)
@@ -1,4 +1,4 @@
 <?xml version="1.0"?>
-<robot xmlns:xacro="http://www.ros.org/wiki/xacro">
+<robot xmlns:xacro="http://www.ros.org/wiki/xacro" name="my_rover">
     <xacro:property name="constant"     value = "0.083333333"/> #1/12
     <xacro:property name="mass"         value = "0.5"/>
@@ -21,7 +21,10 @@
             <origin xyz="0.0 0.0 0.0" rpy="0.0 0.0 0.0"/>
             <!-- refer this "urdf/tutorials/adding physical and collision properties into urdf file" page for the equation -->
-            <inertia ixx="${(constant * mass) * (height*height + depth*depth)}" ixy="0.0" ixz="0.0"
-                     iyy="${(constant * mass) * (width*width + depth*depth)}" iyz="0.0"
-                     izz="${(constant * mass) * (width*width + height*height)}"/>
+            <!-- <inertia ixx="${(constant) * (mass * (height*height + depth*depth))}" ixy="0.0" ixz="0.0"
+                     iyy="${(constant) * (mass * (width*width + depth*depth))}" iyz="0.0"
+                     izz="${(constant) * (mass * (width*width + height*height))}"/> -->
+            <inertia ixx="0.007601" ixy="0.0" ixz="0.0"
+                     iyy="0.03009" iyz="0.0"
+                     izz="0.024365"/>
         </inertial>
         <visual>
@@ -88,7 +91,10 @@
                 <mass value="0.5"/>
                 <origin xyz="0.0 0.0 0.0" rpy="0.0 0.0 0.0"/>
-                <inertia ixx="${constant * mass * (3*radius*radius + length*length)}" ixy="0.0" ixz="0.0"
-                        iyy="${constant * mass * (3*radius*radius + length*length)}" iyz="0.0"
-                        izz="${constant * mass * (radius*radius)}" />
+                <!-- <inertia ixx="${constant * mass * ((3*radius*radius) + (length*length))}" ixy="0.0" ixz="0.0"
+                        iyy="${constant * mass * ((3*radius*radius) + (length*length))}" iyz="0.0"
+                        izz="${constant * mass * (radius*radius)}" /> -->
+                <inertia ixx="0.00042" ixy="0.0" ixz="0.0"
+                        iyy="0.00014" iyz="0.0"
+                        izz="0.00063" />
             </inertial>
             <visual>

Commit message: implemented_localisation

File: urdf/lidar.xacro (robot description, xacro)
@@ -11,5 +11,5 @@
         <visual>
             <geometry>
-                <mesh filename="package://mobile_robot/meshes/lds.stl" scale="0.002 0.002 0.002"/>
+                <mesh filename="package://my_4wheel_bot/meshes/lds.stl" scale="0.002 0.002 0.002"/>
             </geometry>
             <material name="">

File: urdf/robot_core.urdf.xacro (robot description, xacro)
@@ -1,9 +1,9 @@
 <?xml version="1.0"?>
 <robot xmlns:xacro="http://www.ros.org/wiki/xacro" name="my_rover">
-    <xacro:include filename="$(find mobile_robot)/urdf/rover.urdf.xacro"/>
-    <xacro:include filename="$(find mobile_robot)/urdf/lidar.xacro"/>
-    <xacro:include filename="$(find mobile_robot)/urdf/camera.xacro"/>
-    <xacro:include filename="$(find mobile_robot)/urdf/imu_plugin.xacro"/>
-    <!-- <xacro:include filename="$(find mobile_robot)/description/gazebo_control.xacro"/> -->
+    <xacro:include filename="$(find my_4wheel_bot)/urdf/rover.urdf.xacro"/>
+    <xacro:include filename="$(find my_4wheel_bot)/urdf/lidar.xacro"/>
+    <xacro:include filename="$(find my_4wheel_bot)/urdf/camera.xacro"/>
+    <xacro:include filename="$(find my_4wheel_bot)/urdf/imu_plugin.xacro"/>
+    <!-- <xacro:include filename="$(find my_4wheel_bot)/description/gazebo_control.xacro"/> -->
     <gazebo>
         <plugin name="gazebo_ros_control" filename="libgazebo_ros_control.so">

File: urdf/rover.urdf.xacro (robot description, xacro)
@@ -177,8 +177,8 @@
   </xacro:macro>
     <!-- wheel creating using macros -->
-    <!-- <xacro:wheel name = "front_left" path ="package://mobile_robot/meshes/right_tire.stl" x = "0.2" y = "0.25"/>
-    <xacro:wheel name = "front_right" path ="package://mobile_robot/meshes/left_tire.stl" x = "0.2" y = "-0.25"/>
-    <xacro:wheel name = "rear_left" path ="package://mobile_robot/meshes/right_tire.stl" x = "-0.2" y = "0.25"/>
-    <xacro:wheel name = "rear_right" path ="package://mobile_robot/meshes/left_tire.stl" x = "-0.2" y = "-0.25"/> -->
+    <!-- <xacro:wheel name = "front_left" path ="package://my_4wheel_bot/meshes/right_tire.stl" x = "0.2" y = "0.25"/>
+    <xacro:wheel name = "front_right" path ="package://my_4wheel_bot/meshes/left_tire.stl" x = "0.2" y = "-0.25"/>
+    <xacro:wheel name = "rear_left" path ="package://my_4wheel_bot/meshes/right_tire.stl" x = "-0.2" y = "0.25"/>
+    <xacro:wheel name = "rear_right" path ="package://my_4wheel_bot/meshes/left_tire.stl" x = "-0.2" y = "-0.25"/> -->
     <xacro:wheel name = "front_left"    x = "0.2"     y = "0.25"/>
     <xacro:wheel name = "front_right"   x = "0.2"     y = "-0.25"/>
