Commit message: trying to generate the map

File: urdf/rover.urdf.xacro (robot description, xacro)
@@ -28,5 +28,4 @@
         <child link="Chassis"/>
         <origin xyz="0.0 0.0 0.0" rpy="0.0 0.0 0.0"/>
-        <axis xyz="0.0 0.0 0.0"/>
     </joint>
     <link name="Chassis">

Commit message: minor changes

File: urdf/rover.urdf.xacro (robot description, xacro)
@@ -14,6 +14,6 @@
         </inertial>
     </xacro:macro> -->
-    <!-- rover base link -->
-    <link name="base_link">
+    <!-- Dummy_link -->
+    <link name="base_footprint">
     </link>
     <joint name="base_footprint_joint" type="fixed">
@@ -22,5 +22,6 @@
         <origin xyz="0.0 0.0 0.0" rpy="0.0 0.0 0.0"/>
     </joint>
-    <link name="base_footprint">
+    <!-- rover base link -->
+    <link name="base_link">
     </link>
     <joint name="Chassis_joint" type="fixed">

Commit message: Done Navigation

File: urdf/rover.urdf.xacro (robot description, xacro)
@@ -2,24 +2,10 @@
 <robot xmlns:xacro="http://www.ros.org/wiki/xacro" name="my_rover">
     <xacro:property name="constant"     value = "0.083333333"/> #1/12
-    <xacro:property name="mass"         value = "0.5"/>
+    <xacro:property name="mass"         value = "5"/>
     <xacro:property name="width"        value = "0.75"/>
     <xacro:property name="height"       value = "0.15"/>
     <xacro:property name="depth"        value = "0.4"/>
-    <xacro:property name="radius"        value = "0.033"/>
-    <xacro:property name="length"        value = "0.018"/>
-    <!-- <xacro:macro name="default_inertial" params="mass">
-        <inertial>
-            <mass value="${mass}" />
-            <inertia ixx="1.0" ixy="0.0" ixz="0.0" iyy="1.0" iyz="0.0" izz="1.0" />
-        </inertial>
-    </xacro:macro> -->
-    <!-- Dummy_link -->
-    <!-- <link name="base_footprint">
-    </link>
-    <joint name="base_footprint_joint" type="fixed">
-        <parent link="base_link"/>
-        <child link="base_footprint"/>
-        <origin xyz="0.0 0.0 0.0" rpy="0.0 0.0 0.0"/>
-    </joint> -->
+    <xacro:property name="wheel_radius" value = "0.15"/>
+    <xacro:property name="wheel_length" value = "0.1"/>
     <!-- rover base link -->
     <link name="base_link">
@@ -32,7 +18,7 @@
     <link name="Chassis">
         <visual>
-            <origin xyz="0.0 0.0 0.15" rpy="0.0 0.0 0.0"/>
+            <origin xyz="0.0 0.0 ${height}" rpy="0.0 0.0 0.0"/>
             <geometry>
-                <box size="0.75 0.4 0.15" />
+                <box size="${width} ${depth} ${height}" />
             </geometry>
             <material name="">
@@ -41,14 +27,11 @@
         </visual>
         <collision>
-            <origin xyz="0.0 0.0 0.15" rpy="0.0 0.0 0.0"/>
+            <origin xyz="0.0 0.0 ${height}" rpy="0.0 0.0 0.0"/>
             <geometry>
-                <box size="0.75 0.4 0.15" />
+                <box size="${width} ${depth} ${height}" />
             </geometry>
         </collision>
         <inertial>
-            <!-- <inertia ixx="${(constant) * (mass * (height*height + depth*depth))}" ixy="0.0" ixz="0.0"
-                iyy="${(constant) * (mass * (width*width + depth*depth))}" iyz="0.0"
-                izz="${(constant) * (mass * (width*width + height*height))}"/> -->
-            <mass value="5"/>
+            <mass value="${mass}"/>
             <inertia ixx="${(constant) * (5 * (height*height + depth*depth))}" ixy="0.0" ixz="0.0"
                     iyy="${(constant) * (5 * (width*width + depth*depth))}" iyz="0.0"
@@ -82,13 +65,9 @@
         <material> Gazebo/Black</material>
     </gazebo>
-    <!-- <joint name="caster_joint" type="continuous">
-        <parent link="Chassis"/>
-        <child link="caster_link"/>
-        <origin xyz="0.2 0 0.15" rpy="0 0 0"/>
-    </joint>
-    <link name="caster_link">
+    <xacro:macro name="wheel" params="name x y">
+    <link name = "${name}_wheel">
         <visual>
             <geometry>
-                <sphere radius="0.05"/>
+                <cylinder length="${wheel_length}" radius="${wheel_radius}"/>
             </geometry>
             <material name="">
@@ -98,47 +77,9 @@
         <collision>
             <geometry>
-                <sphere radius="0.05"/>
-            </geometry>
-        </collision>
-        <inertial>
-        <origin xyz="0 0 0" />
-        <mass value="0.005" />
-        <inertia ixx="0.001" ixy="0.0" ixz="0.0"
-                iyy="0.001" iyz="0.0"
-                izz="0.001" />
-        </inertial>
-    </link>
-    <gazebo reference = "caster_link">
-        <material> Gazebo/Red</material>
-    </gazebo> -->
-    <!-- <xacro:macro name="wheel" params="name path x y"> -->
-    <xacro:macro name="wheel" params="name x y">
-    <link name = "${name}_wheel">
-        <visual>
-            <geometry>
-                <!-- <origin xyz="0.0 0.0 0.0" rpy="0.0 0.0 0.0"/> -->
-                <cylinder length="0.1" radius="0.15"/>
-                <!-- <mesh filename="${path}" scale="0.005 0.005 0.005"/> #length = 0.0182 radius = "0.0330" -->
-            </geometry>
-            <material name="">
-                <color rgba="1.0 0.0 0.0 1.0"/>
-            </material>
-        </visual>
-        <collision>
-            <geometry>
-                <!-- <origin xyz="0.0 0.0 0.0" rpy="-1.57 0.0 0.0"/> -->
-                <cylinder length="0.1" radius="0.15"/>
-                <!-- <mesh filename="${path}" scale="0.005 0.005 0.005"/> #length = 0.018 diameter = "0.066" -->
+                <sphere radius="${wheel_radius}"/>
                 <contact_coefficients mu="1" kp="1e+13" kd="1.0"/>
             </geometry>
         </collision>
         <inertial>
-            <!-- <inertia ixx="${constant * mass * ((3*radius*radius) + (length*length))}" ixy="0.0" ixz="0.0"
-            iyy="${constant * mass * ((3*radius*radius) + (length*length))}" iyz="0.0"
-            izz="${constant * mass * (radius*radius)}" /> -->
-            <!-- <mass value="2.8498940e-02" />
-            <inertia ixx="1.1175580e-05" ixy="-4.2369783e-11" ixz="-5.9381719e-09"
-            iyy="1.1192413e-05" iyz="-1.4400107e-11"
-            izz="2.0712558e-05" />        -->
             <mass value="2" />
             <inertia ixx="0.1291615" ixy="0.0" ixz="0"
@@ -152,6 +93,4 @@
         <origin xyz="${x} ${y} 0.15" rpy="-1.57 0.0 0.0"/>
         <axis xyz="0.0 0.0 1.0"/>
-        <!-- <origin xyz="${x} ${y} 0.15" rpy="0.0 0.0 0.0"/> -->
-        <!-- <axis xyz="0.0 1.0 0.0"/> -->
         <limit effort="10000" velocity="1000"/>
     </joint>
@@ -172,4 +111,5 @@
       <type>transmission_interface/SimpleTransmission</type>
       <actuator name="${name}_wheel_motor">
+        <hardwareInterface>hardware_interface/VelocityJointInterface</hardwareInterface>
         <mechanicalReduction>1</mechanicalReduction>
       </actuator>
@@ -179,9 +119,4 @@
     </transmission>
   </xacro:macro>
-    <!-- wheel creating using macros -->
-    <!-- <xacro:wheel name = "front_left" path ="package://my_4wheel_bot/meshes/right_tire.stl" x = "0.2" y = "0.25"/>
-    <xacro:wheel name = "front_right" path ="package://my_4wheel_bot/meshes/left_tire.stl" x = "0.2" y = "-0.25"/>
-    <xacro:wheel name = "rear_left" path ="package://my_4wheel_bot/meshes/right_tire.stl" x = "-0.2" y = "0.25"/>
-    <xacro:wheel name = "rear_right" path ="package://my_4wheel_bot/meshes/left_tire.stl" x = "-0.2" y = "-0.25"/> -->
     <xacro:wheel name = "front_left"    x = "0.2"     y = "0.25"/>
     <xacro:wheel name = "front_right"   x = "0.2"     y = "-0.25"/>

Commit message: refined the package

File: urdf/rover.urdf.xacro (robot description, xacro)
@@ -66,6 +66,5 @@
         <material> Gazebo/Black</material>
     </gazebo>
-    <xacro:macro name="wheel" params="name x y">
-    <link name = "${name}_wheel">
+    <link name = "front_left_wheel">
         <visual>
             <geometry>
@@ -92,4 +91,224 @@
         </inertial>
     </link>
+    <joint name="front_left_wheel_joint" type="continuous">
+        <parent link="Chassis"/>
+        <child link="front_left_wheel"/>
+        <origin xyz="0.2 0.25 0.15" rpy="-1.57 0.0 0.0"/>
+        <axis xyz="0.0 0.0 1.0"/>
+        <dynamics damping="0"/>
+        <limit effort="10000" velocity="1000"/>
+    </joint>
+    <!-- This block provides the simulator (Gazebo) with information on a few additional
+    physical properties. See http://gazebosim.org/tutorials/?tut=ros_urdf for more-->
+    <gazebo reference="front_left_wheel">
+      <mu1 value="1"/>
+      <mu2 value="1"/>
+      <kp value="1000000.0" />
+      <kd value="100.0" />
+      <slip1 value="0.5" />
+      <slip2 value="0.5" />
+      <material>Gazebo/Red</material>
+    </gazebo>
+    <!-- This block connects the wheel joint to an actuator (motor), which informs both
+    simulation and visualization of the robot -->
+    <transmission name="front_left_wheel_trans">
+      <type>transmission_interface/SimpleTransmission</type>
+      <actuator name="front_left_wheel_motor">
+        <hardwareInterface>hardware_interface/VelocityJointInterface</hardwareInterface>
+        <mechanicalReduction>1</mechanicalReduction>
+      </actuator>
+      <joint name="front_left_wheel_joint">
+        <hardwareInterface>hardware_interface/VelocityJointInterface</hardwareInterface>
+      </joint>
+    </transmission>
+    <!-- front_right_wheel -->
+    <link name = "front_right_wheel">
+        <visual>
+            <geometry>
+                <cylinder length="${wheel_length}" radius="${wheel_radius}"/>
+            </geometry>
+            <material name="">
+                <color rgba="1.0 0.0 0.0 1.0"/>
+            </material>
+        </visual>
+        <collision>
+            <geometry>
+                <sphere radius="${wheel_radius}"/>
+                <contact_coefficients mu="1" kp="1e+13" kd="1.0"/>
+            </geometry>
+        </collision>
+        <inertial>
+            <mass value="${chassis_wheel}" />
+            <inertia ixx="${(constant) * 0.1 * (3*wheel_radius*wheel_radius + wheel_length*wheel_length)}" ixy="0.0" ixz="0.0"
+            iyy="${(constant) * 0.1 * (3*wheel_radius*wheel_radius + wheel_length*wheel_length)}" iyz="0.0"
+            izz="${0.5 * 0.1 * (wheel_radius*wheel_radius)}" /> #1/2
+        </inertial>
+    </link>
+    <joint name="front_right_wheel_joint" type="continuous">
+        <parent link="Chassis"/>
+        <child link="front_right_wheel"/>
+        <origin xyz="0.2 -0.25 0.15" rpy="1.57 0.0 0.0"/>
+        <axis xyz="0.0 0.0 -1.0"/>
+        <dynamics damping="0"/>
+        <limit effort="10000" velocity="1000"/>
+    </joint>
+    <!-- This block provides the simulator (Gazebo) with information on a few additional
+    physical properties. See http://gazebosim.org/tutorials/?tut=ros_urdf for more-->
+    <gazebo reference="front_right_wheel">
+      <mu1 value="1"/>
+      <mu2 value="1"/>
+      <kp value="1000000.0" />
+      <kd value="100.0" />
+      <slip1 value="0.5" />
+      <slip2 value="0.5" />
+      <material>Gazebo/Red</material>
+    </gazebo>
+    <!-- This block connects the wheel joint to an actuator (motor), which informs both
+    simulation and visualization of the robot -->
+    <transmission name="front_right_wheel_trans">
+      <type>transmission_interface/SimpleTransmission</type>
+      <actuator name="front_right_wheel_motor">
+        <hardwareInterface>hardware_interface/VelocityJointInterface</hardwareInterface>
+        <mechanicalReduction>1</mechanicalReduction>
+      </actuator>
+      <joint name="front_right_wheel_joint">
+        <hardwareInterface>hardware_interface/VelocityJointInterface</hardwareInterface>
+      </joint>
+    </transmission>
+    <link name = "rear_left_wheel">
+        <visual>
+            <geometry>
+                <cylinder length="${wheel_length}" radius="${wheel_radius}"/>
+            </geometry>
+            <material name="">
+                <color rgba="1.0 0.0 0.0 1.0"/>
+            </material>
+        </visual>
+        <collision>
+            <geometry>
+                <sphere radius="${wheel_radius}"/>
+                <contact_coefficients mu="1" kp="1e+13" kd="1.0"/>
+            </geometry>
+        </collision>
+        <inertial>
+            <mass value="${chassis_wheel}" />
+            <inertia ixx="${(constant) * 0.1 * (3*wheel_radius*wheel_radius + wheel_length*wheel_length)}" ixy="0.0" ixz="0.0"
+            iyy="${(constant) * 0.1 * (3*wheel_radius*wheel_radius + wheel_length*wheel_length)}" iyz="0.0"
+            izz="${0.5 * 0.1 * (wheel_radius*wheel_radius)}" /> #1/2
+            <!-- <inertia ixx="0.000645833" ixy="0.0" ixz="0"
+            iyy="0.000645833" iyz="0"
+            izz="0.001125" /> -->
+        </inertial>
+    </link>
+    <joint name="rear_left_wheel_joint" type="continuous">
+        <parent link="Chassis"/>
+        <child link="rear_left_wheel"/>
+        <origin xyz="-0.2 0.25 0.15" rpy="-1.57 0.0 0.0"/>
+        <axis xyz="0.0 0.0 1.0"/>
+        <dynamics damping="0"/>
+        <limit effort="10000" velocity="1000"/>
+    </joint>
+    <!-- This block provides the simulator (Gazebo) with information on a few additional
+    physical properties. See http://gazebosim.org/tutorials/?tut=ros_urdf for more-->
+    <gazebo reference="rear_left_wheel">
+      <mu1 value="1"/>
+      <mu2 value="1"/>
+      <kp value="1000000.0" />
+      <kd value="100.0" />
+      <slip1 value="0.5" />
+      <slip2 value="0.5" />
+      <material>Gazebo/Red</material>
+    </gazebo>
+    <!-- This block connects the wheel joint to an actuator (motor), which informs both
+    simulation and visualization of the robot -->
+    <transmission name="rear_left_wheel_trans">
+      <type>transmission_interface/SimpleTransmission</type>
+      <actuator name="rear_left_wheel_motor">
+        <hardwareInterface>hardware_interface/VelocityJointInterface</hardwareInterface>
+        <mechanicalReduction>1</mechanicalReduction>
+      </actuator>
+      <joint name="rear_left_wheel_joint">
+        <hardwareInterface>hardware_interface/VelocityJointInterface</hardwareInterface>
+      </joint>
+    </transmission>
+    <link name = "rear_right_wheel">
+        <visual>
+            <geometry>
+                <cylinder length="${wheel_length}" radius="${wheel_radius}"/>
+            </geometry>
+            <material name="">
+                <color rgba="1.0 0.0 0.0 1.0"/>
+            </material>
+        </visual>
+        <collision>
+            <geometry>
+                <sphere radius="${wheel_radius}"/>
+                <contact_coefficients mu="1" kp="1e+13" kd="1.0"/>
+            </geometry>
+        </collision>
+        <inertial>
+            <mass value="${chassis_wheel}" />
+            <inertia ixx="${(constant) * 0.1 * (3*wheel_radius*wheel_radius + wheel_length*wheel_length)}" ixy="0.0" ixz="0.0"
+            iyy="${(constant) * 0.1 * (3*wheel_radius*wheel_radius + wheel_length*wheel_length)}" iyz="0.0"
+            izz="${0.5 * 0.1 * (wheel_radius*wheel_radius)}" /> #1/2
+            <!-- <inertia ixx="0.000645833" ixy="0.0" ixz="0"
+            iyy="0.000645833" iyz="0"
+            izz="0.001125" /> -->
+        </inertial>
+    </link>
+    <joint name="rear_right_wheel_joint" type="continuous">
+        <parent link="Chassis"/>
+        <child link="rear_right_wheel"/>
+        <origin xyz="-0.2 -0.25 0.15" rpy="1.57 0.0 0.0"/>
+        <axis xyz="0.0 0.0 -1.0"/>
+        <dynamics damping="0"/>
+        <limit effort="10000" velocity="1000"/>
+    </joint>
+    <!-- This block provides the simulator (Gazebo) with information on a few additional
+    physical properties. See http://gazebosim.org/tutorials/?tut=ros_urdf for more-->
+    <gazebo reference="rear_right_wheel">
+      <mu1 value="1"/>
+      <mu2 value="1"/>
+      <kp value="1000000.0" />
+      <kd value="100.0" />
+      <slip1 value="0.5" />
+      <slip2 value="0.5" />
+      <material>Gazebo/Red</material>
+    </gazebo>
+    <!-- This block connects the wheel joint to an actuator (motor), which informs both
+    simulation and visualization of the robot -->
+    <transmission name="rear_right_wheel_trans">
+      <type>transmission_interface/SimpleTransmission</type>
+      <actuator name="rear_right_wheel_motor">
+        <hardwareInterface>hardware_interface/VelocityJointInterface</hardwareInterface>
+        <mechanicalReduction>1</mechanicalReduction>
+      </actuator>
+      <joint name="rear_right_wheel_joint">
+        <hardwareInterface>hardware_interface/VelocityJointInterface</hardwareInterface>
+      </joint>
+    </transmission>
+    <!-- <xacro:macro name="wheel" params="name x y">
+    <link name = "${name}_wheel">
+        <visual>
+            <geometry>
+                <cylinder length="${wheel_length}" radius="${wheel_radius}"/>
+            </geometry>
+            <material name="">
+                <color rgba="1.0 0.0 0.0 1.0"/>
+            </material>
+        </visual>
+        <collision>
+            <geometry>
+                <sphere radius="${wheel_radius}"/>
+                <contact_coefficients mu="1" kp="1e+13" kd="1.0"/>
+            </geometry>
+        </collision>
+        <inertial>
+            <mass value="${chassis_wheel}" />
+            <inertia ixx="${(constant) * 0.1 * (3*wheel_radius*wheel_radius + wheel_length*wheel_length)}" ixy="0.0" ixz="0.0"
+            iyy="${(constant) * 0.1 * (3*wheel_radius*wheel_radius + wheel_length*wheel_length)}" iyz="0.0"
+            izz="${0.5 * 0.1 * (wheel_radius*wheel_radius)}" /> #1/2
+        </inertial>
+    </link>
     <joint name="${name}_wheel_joint" type="continuous">
         <parent link="Chassis"/>
@@ -100,6 +319,4 @@
         <limit effort="10000" velocity="1000"/>
     </joint>
-    <!-- This block provides the simulator (Gazebo) with information on a few additional
-    physical properties. See http://gazebosim.org/tutorials/?tut=ros_urdf for more-->
     <gazebo reference="${name}_wheel">
       <mu1 value="1"/>
@@ -111,6 +328,4 @@
       <material>Gazebo/Red</material>
     </gazebo>
-    <!-- This block connects the wheel joint to an actuator (motor), which informs both
-    simulation and visualization of the robot -->
     <transmission name="${name}_wheel_trans">
       <type>transmission_interface/SimpleTransmission</type>
@@ -127,4 +342,4 @@
     <xacro:wheel name = "front_right"   x = "0.2"     y = "-0.25"/>
     <xacro:wheel name = "rear_left"     x = "-0.2"    y = "0.25"/>
-    <xacro:wheel name = "rear_right"    x = "-0.2"    y = "-0.25"/>
+    <xacro:wheel name = "rear_right"    x = "-0.2"    y = "-0.25"/> -->
 </robot>
