Commit message: almost made the bot move

File: description/gazebo_control.xacro (robot description, xacro)
@@ -2,15 +2,13 @@
 <robot xmlns:xacro="http://www.ros.org/wiki/xacro">
     <gazebo>
-        <plugin filename = "libgazebo_ros_diff_drive.so" name = "diff_drive">
+        <plugin filename = "libgazebo_ros_diff_drive.so" name = "differential_drive_controller">
             <!-- wheel info -->
-            <!-- <front_left_joint>front_left_wheel_joint</front_left_joint>
-            <front_right_joint>front_right_wheel_joint</front_right_joint>
-            <rear_left_joint>rear_left_wheel_joint</rear_left_joint>
-            <rear_right_joint>rear_right_wheel_joint</rear_right_joint> -->
-            <leftJoint> front_left_wheel_joint </leftJoint>
-            <rightJoint> front_right_wheel_joint </rightJoint>
+            <leftFrontJoint>front_left_wheel_joint</leftFrontJoint>
+            <rightFrontJoint>front_right_wheel_joint</rightFrontJoint>
+            <leftRearJoint>rear_left_wheel_joint</leftRearJoint>
+            <rightRearJoint>rear_right_wheel_joint</rightRearJoint>
+            <!-- <leftJoint> front_left_wheel_joint </leftJoint>
+            <rightJoint> front_right_wheel_joint </rightJoint> -->
             <wheelSeparation>0.4</wheelSeparation>
-            <!-- <front_wheel_seperation>0.4</front_wheel_seperation>
-            <rear_wheel_seperation>0,4</rear_wheel_seperation> -->
             <wheelDiameter>0.066</wheelDiameter>
             <!-- limits -->
@@ -22,7 +20,7 @@
             <odometrySource>1</odometrySource>
             <commandTopic>cmd_vel</commandTopic>
-            <robotBaseFrame>Chassis</robotBaseFrame>
+            <robotBaseFrame>world</robotBaseFrame>
             <!-- output -->
-            <updateRate>1</updateRate>
+            <updateRate>50.0</updateRate>
             <publish_odom>true</publish_odom>
             <publishTf>1</publishTf>
@@ -30,4 +28,5 @@
             <publishWheelTF>true</publishWheelTF>
             <publishWheelJointState>true</publishWheelJointState>
+            <legacyMode>false</legacyMode>
         </plugin>
     </gazebo>

File: urdf/lidar.xacro (robot description, xacro)
@@ -30,12 +30,14 @@
                     izz="0.00005" />
         </inertial>
-        <sensor name = "laser" type = "ray">
+    </link>
+    <gazebo reference = "lidar_link">
+        <sensor name = "head_hokuyo_sensor" type = "ray">
             <pose> 0 0 0 0 0 0 </pose>
             <visualize>true</visualize>
-            <update_rate>10</update_rate>
+            <update_rate>50</update_rate>
             <ray>
                 <scan>
                     <horizontal>
-                        <samples>360</samples>
+                        <samples>720</samples>
                         <resolution>1</resolution>
                         <min_angle>-2.356194</min_angle>  <!-- -135 degrees in radians -->
@@ -44,19 +46,19 @@
                 </scan>
                 <range>
-                    <min>0.02</min>   <!-- Minimum range in meters -->
-                    <max>15.0</max>   <!-- Maximum range in meters -->
+                    <min>0.3</min>   <!-- Minimum range in meters -->
+                    <max>15</max>   <!-- Maximum range in meters -->
                     <resolution>0.01</resolution>   <!-- Range resolution in meters -->
                 </range>
             </ray>
-            <plugin name="laser" filename="libgazebo_ros_ray_sensor.so">
-                <ros>
-                    <argument>~/out:=scan</argument>
+            <plugin name="gazebo_ros_head_hokuyo_controller" filename="libgazebo_ros_laser.so">
+                <!-- <robotNamespace>my_rover</robotNamespace> -->
+                <topicName>/scan</topicName>
+                <!-- <ros>
+                    <remapping>~/out:=scan</remapping>
                 </ros>
-                <output_type>sensor_msgs/LaserScan</output_type>
-                <frame_name>lidar_link</frame_name>
+                <output_type>sensor_msgs/LaserScan</output_type> -->
+                <frameName>lidar_link</frameName>
             </plugin>
         </sensor>
-    </link>
-    <gazebo reference = "lidar_link">
         <material> Gazebo/Blue </material>
     </gazebo>

File: urdf/rover.urdf.xacro (robot description, xacro)
@@ -19,5 +19,5 @@
         <inertial>
             <mass value="0.5"/>
-            <origin xyz="0.0 0.0 0.0" rpy="0.0 0.0 0.0"/>
+            <origin xyz="0.0 0.0 0.135" rpy="0.0 0.0 0.0"/>
             <!-- refer this "urdf/tutorials/adding physical and collision properties into urdf file" page for the equation -->
             <!-- <inertia ixx="${(constant) * (mass * (height*height + depth*depth))}" ixy="0.0" ixz="0.0"
@@ -109,5 +109,5 @@
                 <origin xyz="0.0 0.0 0.0" rpy="0.0 0.0 0.0"/>
                 <geometry>
-                    <mesh filename="${path}" scale="0.005 0.005 0.005"/>
+                    <cylinder radius="${radius}" length="${length}"/>
                 </geometry>
             </collision>
@@ -115,5 +115,18 @@
         <gazebo reference = "${name}_wheel">
             <material> Gazebo/Red </material>
+            <mu1 value="200.0"/>
+            <mu2 value="100.0"/>
+            <kp value="10000000.0" />
+            <kd value="1.0" />
         </gazebo>
+        <transmission name="${name}_wheel_trans">
+            <type>transmission_interface/SimpleTransmission</type>
+            <actuator name="${name}_wheel_motor">
+                <mechanicalReduction>1</mechanicalReduction>
+            </actuator>
+            <joint name="${name}_wheel_joint">
+                <hardwareInterface>hardware_interface/VelocityJointInterface</hardwareInterface>
+            </joint>
+        </transmission>
     </xacro:macro>
     <!-- wheel creating using macros -->

Commit message: some minor changes

File: description/gazebo_control.xacro (robot description, xacro)
@@ -4,10 +4,10 @@
         <plugin filename = "libgazebo_ros_diff_drive.so" name = "differential_drive_controller">
             <!-- wheel info -->
-            <leftFrontJoint>front_left_wheel_joint</leftFrontJoint>
+            <!-- <leftFrontJoint>front_left_wheel_joint</leftFrontJoint>
             <rightFrontJoint>front_right_wheel_joint</rightFrontJoint>
             <leftRearJoint>rear_left_wheel_joint</leftRearJoint>
-            <rightRearJoint>rear_right_wheel_joint</rightRearJoint>
-            <!-- <leftJoint> front_left_wheel_joint </leftJoint>
-            <rightJoint> front_right_wheel_joint </rightJoint> -->
+            <rightRearJoint>rear_right_wheel_joint</rightRearJoint> -->
+            <leftJoint> ['front_left_wheel_joint', 'rear_left_wheel_joint'] </leftJoint>
+            <rightJoint> ['front_right_wheel_joint', 'rear_right_wheel_joint'] </rightJoint>
             <wheelSeparation>0.4</wheelSeparation>
             <wheelDiameter>0.066</wheelDiameter>

File: urdf/rover.urdf.xacro (robot description, xacro)
@@ -13,5 +13,5 @@
         <parent link="world"/>
         <child link="Chassis"/>
-        <origin xyz="0.0 0.0 0.135" rpy="0.0 0.0 0.0"/>
+        <origin xyz="0.0 0.0 0.165" rpy="0.0 0.0 0.0"/>
         <axis xyz="0.0 0.0 0.0"/>
     </joint>
@@ -19,5 +19,5 @@
         <inertial>
             <mass value="0.5"/>
-            <origin xyz="0.0 0.0 0.135" rpy="0.0 0.0 0.0"/>
+            <origin xyz="0.0 0.0 0.165" rpy="0.0 0.0 0.0"/>
             <!-- refer this "urdf/tutorials/adding physical and collision properties into urdf file" page for the equation -->
             <!-- <inertia ixx="${(constant) * (mass * (height*height + depth*depth))}" ixy="0.0" ixz="0.0"
@@ -86,4 +86,5 @@
             <origin xyz="${x} ${y} 0.0" rpy="0.0 0.0 0.0"/>
             <axis xyz="0.0 1.0 0.0"/>
+            <limit effort="100.0" lower="-3.14159" upper="3.14159" velocity="6.0"/>
         </joint>
         <link name="${name}_wheel">
@@ -115,6 +116,6 @@
         <gazebo reference = "${name}_wheel">
             <material> Gazebo/Red </material>
-            <mu1 value="200.0"/>
-            <mu2 value="100.0"/>
+            <mu1 value="0.001"/>
+            <mu2 value="0.001"/>
             <kp value="10000000.0" />
             <kd value="1.0" />
@@ -131,7 +132,7 @@
     </xacro:macro>
     <!-- wheel creating using macros -->
-    <xacro:wheel name = "front_left" path ="package://mobile_robot/meshes/right_tire.stl" x = "0.187" y = "0.25"/>
-    <xacro:wheel name = "front_right" path ="package://mobile_robot/meshes/left_tire.stl" x = "0.187" y = "-0.25"/>
-    <xacro:wheel name = "rear_left" path ="package://mobile_robot/meshes/right_tire.stl" x = "-0.187" y = "0.25"/>
-    <xacro:wheel name = "rear_right" path ="package://mobile_robot/meshes/left_tire.stl" x = "-0.187" y = "-0.25"/>
+    <xacro:wheel name = "front_left" path ="package://mobile_robot/meshes/right_tire.stl" x = "0.187" y = "0.245"/>
+    <xacro:wheel name = "front_right" path ="package://mobile_robot/meshes/left_tire.stl" x = "0.187" y = "-0.245"/>
+    <xacro:wheel name = "rear_left" path ="package://mobile_robot/meshes/right_tire.stl" x = "-0.187" y = "0.245"/>
+    <xacro:wheel name = "rear_right" path ="package://mobile_robot/meshes/left_tire.stl" x = "-0.187" y = "-0.245"/>
 </robot>

Commit message: Bot moving

File: description/gazebo_control.xacro (robot description, xacro)
@@ -8,6 +8,6 @@
             <leftRearJoint>rear_left_wheel_joint</leftRearJoint>
             <rightRearJoint>rear_right_wheel_joint</rightRearJoint> -->
-            <leftJoint> ['front_left_wheel_joint', 'rear_left_wheel_joint'] </leftJoint>
-            <rightJoint> ['front_right_wheel_joint', 'rear_right_wheel_joint'] </rightJoint>
+            <leftJoint> [left_wheel_joint'] </leftJoint>
+            <rightJoint> ['right_wheel_joint'] </rightJoint>
             <wheelSeparation>0.4</wheelSeparation>
             <wheelDiameter>0.066</wheelDiameter>
@@ -20,5 +20,5 @@
             <odometrySource>1</odometrySource>
             <commandTopic>cmd_vel</commandTopic>
-            <robotBaseFrame>world</robotBaseFrame>
+            <robotBaseFrame>base_link</robotBaseFrame>
             <!-- output -->
             <updateRate>50.0</updateRate>

File: urdf/rover.urdf (robot description, URDF)
Before this commit: robot my_rover, 7 links, 6 joints
Links:
- removed link lidar_link
Joints:
- removed joint lidar_joint

File: urdf/rover.urdf.xacro (robot description, xacro)
@@ -8,25 +8,21 @@
     <xacro:property name="radius"        value = "0.033"/>
     <xacro:property name="length"        value = "0.018"/>
+    <!-- <xacro:macro name="default_inertial" params="mass">
+        <inertial>
+            <mass value="${mass}" />
+            <inertia ixx="1.0" ixy="0.0" ixz="0.0" iyy="1.0" iyz="0.0" izz="1.0" />
+        </inertial>
+    </xacro:macro> -->
     <!-- rover base link -->
-    <link name="world"/>
+    <!-- <link name="world"/>
     <joint name="Chassis_joint" type="fixed">
         <parent link="world"/>
-        <child link="Chassis"/>
+        <child link="base_link"/>
         <origin xyz="0.0 0.0 0.165" rpy="0.0 0.0 0.0"/>
         <axis xyz="0.0 0.0 0.0"/>
-    </joint>
-    <link name="Chassis">
-        <inertial>
-            <mass value="0.5"/>
-            <origin xyz="0.0 0.0 0.165" rpy="0.0 0.0 0.0"/>
-            <!-- refer this "urdf/tutorials/adding physical and collision properties into urdf file" page for the equation -->
-            <!-- <inertia ixx="${(constant) * (mass * (height*height + depth*depth))}" ixy="0.0" ixz="0.0"
-                     iyy="${(constant) * (mass * (width*width + depth*depth))}" iyz="0.0"
-                     izz="${(constant) * (mass * (width*width + height*height))}"/> -->
-            <inertia ixx="0.007601" ixy="0.0" ixz="0.0"
-                     iyy="0.03009" iyz="0.0"
-                     izz="0.024365"/>
-        </inertial>
+    </joint> -->
+    <link name="base_link">
         <visual>
+            <origin xyz="0.0 0.0 0.15" rpy="0.0 0.0 0.0"/>
             <geometry>
                 <box size="0.75 0.4 0.15" />
@@ -37,28 +33,30 @@
         </visual>
         <collision>
-            <origin xyz="0.0 0.0 0.0" rpy="0.0 0.0 0.0"/>
+            <origin xyz="0.0 0.0 0.15" rpy="0.0 0.0 0.0"/>
             <geometry>
                 <box size="0.75 0.4 0.15" />
             </geometry>
         </collision>
+        <inertial>
+            <!-- <inertia ixx="${(constant) * (mass * (height*height + depth*depth))}" ixy="0.0" ixz="0.0"
+                iyy="${(constant) * (mass * (width*width + depth*depth))}" iyz="0.0"
+                izz="${(constant) * (mass * (width*width + height*height))}"/> -->
+            <origin xyz="0.0 0.0 0.0" rpy="0.0 0.0 0.0"/>
+            <mass value="10"/>
+            <inertia ixx="${(constant) * (10 * (height*height + depth*depth))}" ixy="0.0" ixz="0.0"
+                    iyy="${(constant) * (10 * (width*width + depth*depth))}" iyz="0.0"
+                    izz="${(constant) * (10 * (width*width + height*height))}"/>
+        </inertial>
     </link>
-    <gazebo reference = "Chassis">
+    <gazebo reference = "base_link">
         <material> Gazebo/Orange </material>
     </gazebo>
-        <!-- camera/sensor mount -->
-    <joint name="mount_joint" type="fixed">
-        <parent link="Chassis"/>
+        <joint name="mount_joint" type="fixed">
+        <parent link="base_link"/>
         <child link="mount_link"/>
-        <origin xyz="0.2 0.0 0.124" rpy="0.0 0.0 0.0"/>
+        <origin xyz="0.2 0.0 0.25" rpy="0.0 0.0 0.0"/>
         <axis xyz="0.0 0.0 0.0"/>
     </joint>
     <link name="mount_link">
-        <inertial>
-            <mass value="0.0"/>
-            <origin xyz="0.0 0.0 0.0" rpy="0.0 0.0 0.0"/>
-            <inertia ixx="0.0" ixy="0.0" ixz="0.0"
-                    iyy="0.0" iyz="0.0"
-                    izz="0.0" />
-        </inertial>
         <visual>
             <geometry>
@@ -70,5 +68,4 @@
         </visual>
         <collision>
-            <origin xyz="0.0 0.0 0.0" rpy="0.0 0.0 0.0"/>
             <geometry>
                 <cylinder radius="0.08" length="0.1"/>
@@ -79,56 +76,60 @@
         <material> Gazebo/Black</material>
     </gazebo>
-    <!-- defining xacro style for repeating elements -->
-    <xacro:macro name="wheel" params="name path x y">
-        <joint name="${name}_wheel_joint" type="continuous">
-            <parent link="Chassis"/>
-            <child link="${name}_wheel"/>
-            <origin xyz="${x} ${y} 0.0" rpy="0.0 0.0 0.0"/>
-            <axis xyz="0.0 1.0 0.0"/>
-            <limit effort="100.0" lower="-3.14159" upper="3.14159" velocity="6.0"/>
-        </joint>
-        <link name="${name}_wheel">
-            <inertial>
-                <mass value="0.5"/>
-                <origin xyz="0.0 0.0 0.0" rpy="0.0 0.0 0.0"/>
-                <!-- <inertia ixx="${constant * mass * ((3*radius*radius) + (length*length))}" ixy="0.0" ixz="0.0"
-                        iyy="${constant * mass * ((3*radius*radius) + (length*length))}" iyz="0.0"
-                        izz="${constant * mass * (radius*radius)}" /> -->
-                <inertia ixx="0.00042" ixy="0.0" ixz="0.0"
-                        iyy="0.00014" iyz="0.0"
-                        izz="0.00063" />
-            </inertial>
-            <visual>
-                <geometry>
-                    <mesh filename="${path}" scale="0.005 0.005 0.005"/> #length = 0.018 radius = "0.066"
-                </geometry>
-                <material name="">
-                    <color rgba="1.0 0.0 0.0 1.0"/>
-                </material>
-            </visual>
-            <collision>
-                <origin xyz="0.0 0.0 0.0" rpy="0.0 0.0 0.0"/>
-                <geometry>
-                    <cylinder radius="${radius}" length="${length}"/>
-                </geometry>
-            </collision>
-        </link>
-        <gazebo reference = "${name}_wheel">
-            <material> Gazebo/Red </material>
-            <mu1 value="0.001"/>
-            <mu2 value="0.001"/>
-            <kp value="10000000.0" />
-            <kd value="1.0" />
-        </gazebo>
-        <transmission name="${name}_wheel_trans">
-            <type>transmission_interface/SimpleTransmission</type>
-            <actuator name="${name}_wheel_motor">
-                <mechanicalReduction>1</mechanicalReduction>
-            </actuator>
-            <joint name="${name}_wheel_joint">
-                <hardwareInterface>hardware_interface/VelocityJointInterface</hardwareInterface>
-            </joint>
-        </transmission>
-    </xacro:macro>
+  <xacro:macro name="wheel" params="name path x y">
+    <link name = "${name}_wheel">
+        <visual>
+            <origin xyz="0.0 0.0 0.0" rpy="0.0 0.0 0.0"/>
+            <geometry>
+                <mesh filename="${path}" scale="0.005 0.005 0.005"/> #length = 0.018 radius = "0.066"
+            </geometry>
+            <material name="">
+                <color rgba="1.0 0.0 0.0 1.0"/>
+            </material>
+        </visual>
+        <collision>
+            <origin xyz="0.0 0.0 0.0" rpy="0.0 0.0 0.0"/>
+            <geometry>
+                <mesh filename="${path}" scale="0.005 0.005 0.005"/> #length = 0.018 radius = "0.066"
+            </geometry>
+        </collision>
+        <inertial>
+            <!-- <inertia ixx="${constant * mass * ((3*radius*radius) + (length*length))}" ixy="0.0" ixz="0.0"
+            iyy="${constant * mass * ((3*radius*radius) + (length*length))}" iyz="0.0"
+            izz="${constant * mass * (radius*radius)}" /> -->
+            <origin xyz="0.0 0.0 0.0" rpy="0.0 0.0 0.0"/>
+            <mass value="1"/>
+            <inertia ixx="${constant * 1 * ((3*radius*radius) + (length*length))}" ixy="0.0" ixz="0.0"
+                    iyy="${constant * 1 * ((3*radius*radius) + (length*length))}" iyz="0.0"
+                    izz="${constant * 1 * (radius*radius)}"/>
+        </inertial>
+    </link>
+    <joint name="${name}_wheel_joint" type="continuous">
+        <parent link="base_link"/>
+        <child link="${name}_wheel"/>
+        <origin xyz="${x} ${y} 0.15" rpy="0.0 0.0 0.0"/>
+        <axis xyz="0.0 1.0 0.0"/>
+        <!-- <limit effort="100.0" lower="-3.14159" upper="3.14159" velocity="6.0"/>  -->
+    </joint>
+    <!-- This block provides the simulator (Gazebo) with information on a few additional
+    physical properties. See http://gazebosim.org/tutorials/?tut=ros_urdf for more-->
+    <gazebo reference="${name}_wheel">
+      <mu1 value="200.0"/>
+      <mu2 value="100.0"/>
+      <kp value="10000000.0" />
+      <kd value="1.0" />
+      <material>Gazebo/Red</material>
+    </gazebo>
+    <!-- This block connects the wheel joint to an actuator (motor), which informs both
+    simulation and visualization of the robot -->
+    <transmission name="${name}_wheel_trans">
+      <type>transmission_interface/SimpleTransmission</type>
+      <actuator name="${name}_wheel_motor">
+        <mechanicalReduction>1</mechanicalReduction>
+      </actuator>
+      <joint name="${name}_wheel_joint">
+        <hardwareInterface>hardware_interface/VelocityJointInterface</hardwareInterface>
+      </joint>
+    </transmission>
+  </xacro:macro>
     <!-- wheel creating using macros -->
     <xacro:wheel name = "front_left" path ="package://mobile_robot/meshes/right_tire.stl" x = "0.187" y = "0.245"/>
