Commit message: almost there in generating map

File: description/gazebo_control.xacro (robot description, xacro)
@@ -1,4 +1,4 @@
 <?xml version="1.0"?>
-<robot xmlns:xacro="http://www.ros.org/wiki/xacro">
+<robot xmlns:xacro="http://www.ros.org/wiki/xacro" name = "my_rover">
     <gazebo>
         <plugin filename = "libgazebo_ros_diff_drive.so" name = "differential_drive_controller">
@@ -8,6 +8,6 @@
             <leftRearJoint>rear_left_wheel_joint</leftRearJoint>
             <rightRearJoint>rear_right_wheel_joint</rightRearJoint> -->
-            <leftJoint> [left_wheel_joint'] </leftJoint>
-            <rightJoint> ['right_wheel_joint'] </rightJoint>
+            <leftJoint> ['front_left_wheel_joint', 'rear_left_wheel_joint'] </leftJoint>
+            <rightJoint> ['front_right_wheel_joint', 'rear_right_wheel_joint'] </rightJoint>
             <wheelSeparation>0.4</wheelSeparation>
             <wheelDiameter>0.066</wheelDiameter>
@@ -20,5 +20,5 @@
             <odometrySource>1</odometrySource>
             <commandTopic>cmd_vel</commandTopic>
-            <robotBaseFrame>base_link</robotBaseFrame>
+            <robotBaseFrame>Chassis</robotBaseFrame>
             <!-- output -->
             <updateRate>50.0</updateRate>

File: urdf/lidar.xacro (robot description, xacro)
@@ -34,5 +34,5 @@
         <sensor name = "head_hokuyo_sensor" type = "ray">
             <pose> 0 0 0 0 0 0 </pose>
-            <visualize>true</visualize>
+            <visualize>false</visualize>
             <update_rate>50</update_rate>
             <ray>
@@ -41,11 +41,11 @@
                         <samples>720</samples>
                         <resolution>1</resolution>
-                        <min_angle>-2.356194</min_angle>  <!-- -135 degrees in radians -->
-                        <max_angle>2.356194</max_angle>   <!-- 135 degrees in radians -->
+                        <min_angle>-3.14159</min_angle>  <!-- -135 degrees in radians -->
+                        <max_angle>3.14159</max_angle>   <!-- 135 degrees in radians -->
                     </horizontal>
                 </scan>
                 <range>
                     <min>0.3</min>   <!-- Minimum range in meters -->
-                    <max>15</max>   <!-- Maximum range in meters -->
+                    <max>20</max>   <!-- Maximum range in meters -->
                     <resolution>0.01</resolution>   <!-- Range resolution in meters -->
                 </range>

File: urdf/robot_core.urdf.xacro (robot description, xacro)
@@ -3,4 +3,5 @@
     <xacro:include filename="$(find mobile_robot)/urdf/rover.urdf.xacro"/>
     <xacro:include filename="$(find mobile_robot)/urdf/lidar.xacro"/>
+    <xacro:include filename="$(find mobile_robot)/urdf/camera.xacro"/>
     <!-- <xacro:include filename="$(find mobile_robot)/description/transmission.urdf"/> -->
     <!-- <xacro:include filename="$(find mobile_robot)/description/gazebo_control.xacro"/> -->

File: urdf/rover.urdf.xacro (robot description, xacro)
@@ -15,12 +15,20 @@
     </xacro:macro> -->
     <!-- rover base link -->
-    <!-- <link name="world"/>
+    <link name="base_link">
+    </link>
+    <joint name="base_footprint_joint" type="fixed">
+        <parent link="base_link"/>
+        <child link="base_footprint"/>
+        <origin xyz="0.0 0.0 0.0" rpy="0.0 0.0 0.0"/>
+    </joint>
+    <link name="base_footprint">
+    </link>
     <joint name="Chassis_joint" type="fixed">
-        <parent link="world"/>
-        <child link="base_link"/>
-        <origin xyz="0.0 0.0 0.165" rpy="0.0 0.0 0.0"/>
+        <parent link="base_link"/>
+        <child link="Chassis"/>
+        <origin xyz="0.0 0.0 0.0" rpy="0.0 0.0 0.0"/>
         <axis xyz="0.0 0.0 0.0"/>
-    </joint> -->
-    <link name="base_link">
+    </joint>
+    <link name="Chassis">
         <visual>
             <origin xyz="0.0 0.0 0.15" rpy="0.0 0.0 0.0"/>
@@ -42,19 +50,17 @@
                 iyy="${(constant) * (mass * (width*width + depth*depth))}" iyz="0.0"
                 izz="${(constant) * (mass * (width*width + height*height))}"/> -->
-            <origin xyz="0.0 0.0 0.0" rpy="0.0 0.0 0.0"/>
-            <mass value="10"/>
-            <inertia ixx="${(constant) * (10 * (height*height + depth*depth))}" ixy="0.0" ixz="0.0"
-                    iyy="${(constant) * (10 * (width*width + depth*depth))}" iyz="0.0"
-                    izz="${(constant) * (10 * (width*width + height*height))}"/>
+            <mass value="5"/>
+            <inertia ixx="${(constant) * (5 * (height*height + depth*depth))}" ixy="0.0" ixz="0.0"
+                    iyy="${(constant) * (5 * (width*width + depth*depth))}" iyz="0.0"
+                    izz="${(constant) * (5 * (width*width + height*height))}"/>
         </inertial>
     </link>
-    <gazebo reference = "base_link">
+    <gazebo reference = "Chassis">
         <material> Gazebo/Orange </material>
     </gazebo>
-        <joint name="mount_joint" type="fixed">
-        <parent link="base_link"/>
+    <joint name="mount_joint" type="fixed">
+        <parent link="Chassis"/>
         <child link="mount_link"/>
         <origin xyz="0.2 0.0 0.25" rpy="0.0 0.0 0.0"/>
-        <axis xyz="0.0 0.0 0.0"/>
     </joint>
     <link name="mount_link">
@@ -79,5 +85,4 @@
     <link name = "${name}_wheel">
         <visual>
-            <origin xyz="0.0 0.0 0.0" rpy="0.0 0.0 0.0"/>
             <geometry>
                 <mesh filename="${path}" scale="0.005 0.005 0.005"/> #length = 0.018 radius = "0.066"
@@ -88,5 +93,4 @@
         </visual>
         <collision>
-            <origin xyz="0.0 0.0 0.0" rpy="0.0 0.0 0.0"/>
             <geometry>
                 <mesh filename="${path}" scale="0.005 0.005 0.005"/> #length = 0.018 radius = "0.066"
@@ -97,5 +101,4 @@
             iyy="${constant * mass * ((3*radius*radius) + (length*length))}" iyz="0.0"
             izz="${constant * mass * (radius*radius)}" /> -->
-            <origin xyz="0.0 0.0 0.0" rpy="0.0 0.0 0.0"/>
             <mass value="1"/>
             <inertia ixx="${constant * 1 * ((3*radius*radius) + (length*length))}" ixy="0.0" ixz="0.0"
@@ -105,5 +108,5 @@
     </link>
     <joint name="${name}_wheel_joint" type="continuous">
-        <parent link="base_link"/>
+        <parent link="Chassis"/>
         <child link="${name}_wheel"/>
         <origin xyz="${x} ${y} 0.15" rpy="0.0 0.0 0.0"/>

Commit message: generating map

File: description/gazebo_control.xacro (robot description, xacro)
@@ -3,30 +3,22 @@
     <gazebo>
         <plugin filename = "libgazebo_ros_diff_drive.so" name = "differential_drive_controller">
-            <!-- wheel info -->
-            <!-- <leftFrontJoint>front_left_wheel_joint</leftFrontJoint>
-            <rightFrontJoint>front_right_wheel_joint</rightFrontJoint>
-            <leftRearJoint>rear_left_wheel_joint</leftRearJoint>
-            <rightRearJoint>rear_right_wheel_joint</rightRearJoint> -->
-            <leftJoint> ['front_left_wheel_joint', 'rear_left_wheel_joint'] </leftJoint>
-            <rightJoint> ['front_right_wheel_joint', 'rear_right_wheel_joint'] </rightJoint>
+            <commandTopic>cmd_vel</commandTopic>
+            <odometryTopic>odom</odometryTopic>
+            <odometryFrame>odom</odometryFrame>
+            <odometrySource>world</odometrySource>
+            <publishOdomTF>true</publishOdomTF>
+            <robotBaseFrame>base_link</robotBaseFrame>
+            <publishWheelTF>false</publishWheelTF>
+            <publishTf>true</publishTf>
+            <publishWheelJointState>true</publishWheelJointState>
+            <legacyMode>false</legacyMode>
+            <updateRate>30</updateRate>
+            <leftJoint>rear_left_wheel_joint</leftJoint>
+            <rightJoint>rear_right_wheel_joint</rightJoint>
             <wheelSeparation>0.4</wheelSeparation>
             <wheelDiameter>0.066</wheelDiameter>
-            <!-- limits -->
-            <wheelTorque>100</wheelTorque>
-            <wheelAcceleration> 10.0</wheelAcceleration>
-            <!-- odometry -->
-            <odometryFrame>odom</odometryFrame>
-            <odometryTopic>odom</odometryTopic>
-            <odometrySource>1</odometrySource>
-            <commandTopic>cmd_vel</commandTopic>
-            <robotBaseFrame>Chassis</robotBaseFrame>
-            <!-- output -->
-            <updateRate>50.0</updateRate>
-            <publish_odom>true</publish_odom>
-            <publishTf>1</publishTf>
-            <publishOdomTF>true</publishOdomTF>
-            <publishWheelTF>true</publishWheelTF>
-            <publishWheelJointState>true</publishWheelJointState>
-            <legacyMode>false</legacyMode>
+            <wheelAcceleration>1</wheelAcceleration>
+            <wheelTorque>10</wheelTorque>
+            <rosDebugLevel>na</rosDebugLevel>
         </plugin>
     </gazebo>

File: urdf/lidar.xacro (robot description, xacro)
@@ -11,5 +11,5 @@
         <visual>
             <geometry>
-                <cylinder radius="0.08" length="0.1"/>
+                <mesh filename="package://mobile_robot/meshes/lds.stl" scale="0.002 0.002 0.002"/>
             </geometry>
             <material name="">
@@ -24,13 +24,13 @@
         </collision>
         <inertial>
-            <mass value="0.1"/>
+            <mass value="0.114"/>
             <origin xyz="0.0 0.0 0.0" rpy="0.0 0.0 0.0"/>
-            <inertia ixx="0.00024" ixy="0.0" ixz="0.0"
-                    iyy="0.00024" iyz="0.0"
-                    izz="0.00005" />
+            <inertia ixx="0.001" ixy="0.0" ixz="0.0"
+                    iyy="0.001" iyz="0.0"
+                    izz="0.001" />
         </inertial>
     </link>
     <gazebo reference = "lidar_link">
-        <sensor name = "head_hokuyo_sensor" type = "ray">
+        <sensor name = "lds_lfcd_sensor" type = "ray">
             <pose> 0 0 0 0 0 0 </pose>
             <visualize>false</visualize>
@@ -39,5 +39,5 @@
                 <scan>
                     <horizontal>
-                        <samples>720</samples>
+                        <samples>360</samples>
                         <resolution>1</resolution>
                         <min_angle>-3.14159</min_angle>  <!-- -135 degrees in radians -->
@@ -50,6 +50,11 @@
                     <resolution>0.01</resolution>   <!-- Range resolution in meters -->
                 </range>
+                <noise>
+                    <type>gaussian</type>
+                    <mean>0.0</mean>
+                    <stddev>0.01</stddev>
+                </noise>
             </ray>
-            <plugin name="gazebo_ros_head_hokuyo_controller" filename="libgazebo_ros_laser.so">
+            <plugin name="gazebo_ros_lds_lfcd_controller" filename="libgazebo_ros_laser.so">
                 <!-- <robotNamespace>my_rover</robotNamespace> -->
                 <topicName>/scan</topicName>

File: urdf/robot_core.urdf.xacro (robot description, xacro)
@@ -4,6 +4,5 @@
     <xacro:include filename="$(find mobile_robot)/urdf/lidar.xacro"/>
     <xacro:include filename="$(find mobile_robot)/urdf/camera.xacro"/>
-    <!-- <xacro:include filename="$(find mobile_robot)/description/transmission.urdf"/> -->
-    <!-- <xacro:include filename="$(find mobile_robot)/description/gazebo_control.xacro"/> -->
+    <xacro:include filename="$(find mobile_robot)/urdf/imu_plugin.xacro"/>
     <gazebo>
         <plugin name="gazebo_ros_control" filename="libgazebo_ros_control.so">

File: urdf/rover.urdf.xacro (robot description, xacro)
@@ -17,5 +17,5 @@
     <link name="base_link">
     </link>
-    <joint name="base_footprint_joint" type="fixed">
+    <!-- <joint name="base_footprint_joint" type="fixed">
         <parent link="base_link"/>
         <child link="base_footprint"/>
@@ -23,5 +23,5 @@
     </joint>
     <link name="base_footprint">
-    </link>
+    </link> -->
     <joint name="Chassis_joint" type="fixed">
         <parent link="base_link"/>
@@ -81,9 +81,13 @@
         <material> Gazebo/Black</material>
     </gazebo>
-  <xacro:macro name="wheel" params="name path x y">
-    <link name = "${name}_wheel">
+    <!-- <joint name="caster_joint" type="continuous">
+        <parent link="Chassis"/>
+        <child link="caster_link"/>
+        <origin xyz="0.2 0 0.15" rpy="0 0 0"/>
+    </joint>
+    <link name="caster_link">
         <visual>
             <geometry>
-                <mesh filename="${path}" scale="0.005 0.005 0.005"/> #length = 0.018 radius = "0.066"
+                <sphere radius="0.05"/>
             </geometry>
             <material name="">
@@ -93,5 +97,31 @@
         <collision>
             <geometry>
-                <mesh filename="${path}" scale="0.005 0.005 0.005"/> #length = 0.018 radius = "0.066"
+                <sphere radius="0.05"/>
+            </geometry>
+        </collision>
+        <inertial>
+        <origin xyz="0 0 0" />
+        <mass value="0.005" />
+        <inertia ixx="0.001" ixy="0.0" ixz="0.0"
+                iyy="0.001" iyz="0.0"
+                izz="0.001" />
+        </inertial>
+    </link>
+    <gazebo reference = "caster_link">
+        <material> Gazebo/Red</material>
+    </gazebo> -->
+    <xacro:macro name="wheel" params="name path x y">
+    <link name = "${name}_wheel">
+        <visual>
+            <geometry>
+                <mesh filename="${path}" scale="0.005 0.005 0.005"/> #length = 0.0182 radius = "0.0660"
+            </geometry>
+            <material name="">
+                <color rgba="1.0 0.0 0.0 1.0"/>
+            </material>
+        </visual>
+        <collision>
+            <geometry>
+                <mesh filename="${path}" scale="0.005 0.005 0.005"/> #length = 0.018 diameter = "0.066"
             </geometry>
         </collision>
@@ -100,8 +130,8 @@
             iyy="${constant * mass * ((3*radius*radius) + (length*length))}" iyz="0.0"
             izz="${constant * mass * (radius*radius)}" /> -->
-            <mass value="1"/>
-            <inertia ixx="${constant * 1 * ((3*radius*radius) + (length*length))}" ixy="0.0" ixz="0.0"
-                    iyy="${constant * 1 * ((3*radius*radius) + (length*length))}" iyz="0.0"
-                    izz="${constant * 1 * (radius*radius)}"/>
+            <mass value="2.8498940e-02" />
+            <inertia ixx="1.1175580e-05" ixy="-4.2369783e-11" ixz="-5.9381719e-09"
+            iyy="1.1192413e-05" iyz="-1.4400107e-11"
+            izz="2.0712558e-05" />
         </inertial>
     </link>
@@ -118,5 +148,5 @@
       <mu1 value="200.0"/>
       <mu2 value="100.0"/>
-      <kp value="10000000.0" />
+      <kp value="500000.0" />
       <kd value="1.0" />
       <material>Gazebo/Red</material>

Commit message: map generating

File: description/gazebo_control.xacro (robot description, xacro)
@@ -1,8 +1,9 @@
 <?xml version="1.0"?>
 <robot xmlns:xacro="http://www.ros.org/wiki/xacro" name = "my_rover">
-    <!-- <gazebo>
+    <gazebo>
         <plugin filename = "libgazebo_ros_diff_drive.so" name = "differential_drive_controller">
             <commandTopic>cmd_vel</commandTopic>
             <odometryTopic>odom</odometryTopic>
+            <!-- <num_wheel_pairs> 2 </num_wheel_pairs> -->
             <odometryFrame>odom</odometryFrame>
             <odometrySource>world</odometrySource>
@@ -14,14 +15,16 @@
             <legacyMode>false</legacyMode>
             <updateRate>30</updateRate>
-            <leftJoint>rear_left_wheel_joint</leftJoint>
-            <rightJoint>rear_right_wheel_joint</rightJoint>
-            <wheelSeparation>0.4</wheelSeparation>
-            <wheelDiameter>0.066</wheelDiameter>
+            <leftJoint>front_left_wheel_joint</leftJoint>
+            <rightJoint>front_right_wheel_joint</rightJoint>
+            <!-- <leftJoint>rear_left_wheel_joint</leftJoint> -->
+            <!-- <rightJoint>rear_right_wheel_joint</rightJoint> -->
+            <wheelSeparation>0.5</wheelSeparation>
+            <wheelDiameter>0.3</wheelDiameter>
             <wheelAcceleration>1</wheelAcceleration>
             <wheelTorque>10</wheelTorque>
             <rosDebugLevel>na</rosDebugLevel>
         </plugin>
-    </gazebo> -->
-    <gazebo>
+    </gazebo>
+    <!-- <gazebo>
         <plugin name="skid_steer_drive_controller" filename="libgazebo_ros_skid_steer_drive.so">
             <updateRate>50.0</updateRate>
@@ -43,4 +46,4 @@
             <broadcastTF>false</broadcastTF>
         </plugin>
-    </gazebo>
+    </gazebo> -->
 </robot>

File: urdf/rover.urdf.xacro (robot description, xacro)
@@ -111,9 +111,12 @@
         <material> Gazebo/Red</material>
     </gazebo> -->
-    <xacro:macro name="wheel" params="name path x y">
+    <!-- <xacro:macro name="wheel" params="name path x y"> -->
+    <xacro:macro name="wheel" params="name x y">
     <link name = "${name}_wheel">
         <visual>
             <geometry>
-                <mesh filename="${path}" scale="0.005 0.005 0.005"/> #length = 0.0182 radius = "0.0330"
+                <!-- <origin xyz="0.0 0.0 0.0" rpy="0.0 0.0 0.0"/> -->
+                <cylinder length="0.1" radius="0.15"/>
+                <!-- <mesh filename="${path}" scale="0.005 0.005 0.005"/> #length = 0.0182 radius = "0.0330" -->
             </geometry>
             <material name="">
@@ -123,5 +126,8 @@
         <collision>
             <geometry>
-                <mesh filename="${path}" scale="0.005 0.005 0.005"/> #length = 0.018 diameter = "0.066"
+                <!-- <origin xyz="0.0 0.0 0.0" rpy="-1.57 0.0 0.0"/> -->
+                <cylinder length="0.1" radius="0.15"/>
+                <!-- <mesh filename="${path}" scale="0.005 0.005 0.005"/> #length = 0.018 diameter = "0.066" -->
+                <contact_coefficients mu="1" kp="1e+13" kd="1.0"/>
             </geometry>
         </collision>
@@ -130,8 +136,12 @@
             iyy="${constant * mass * ((3*radius*radius) + (length*length))}" iyz="0.0"
             izz="${constant * mass * (radius*radius)}" /> -->
-            <mass value="2.8498940e-02" />
+            <!-- <mass value="2.8498940e-02" />
             <inertia ixx="1.1175580e-05" ixy="-4.2369783e-11" ixz="-5.9381719e-09"
             iyy="1.1192413e-05" iyz="-1.4400107e-11"
-            izz="2.0712558e-05" />
+            izz="2.0712558e-05" />        -->
+            <mass value="2" />
+            <inertia ixx="0.1291615" ixy="0.0" ixz="0"
+            iyy="0.1291615" iyz="0"
+            izz="0.0374985" />
         </inertial>
     </link>
@@ -139,6 +149,8 @@
         <parent link="Chassis"/>
         <child link="${name}_wheel"/>
-        <origin xyz="${x} ${y} 0.15" rpy="0.0 0.0 0.0"/>
-        <axis xyz="0.0 1.0 0.0"/>
+        <origin xyz="${x} ${y} 0.15" rpy="-1.57 0.0 0.0"/>
+        <axis xyz="0.0 0.0 1.0"/>
+        <!-- <origin xyz="${x} ${y} 0.15" rpy="0.0 0.0 0.0"/> -->
+        <!-- <axis xyz="0.0 1.0 0.0"/> -->
         <!-- <limit effort="100.0" lower="-3.14159" upper="3.14159" velocity="6.0"/>  -->
     </joint>
@@ -165,7 +177,11 @@
   </xacro:macro>
     <!-- wheel creating using macros -->
-    <xacro:wheel name = "front_left" path ="package://mobile_robot/meshes/right_tire.stl" x = "0.187" y = "0.245"/>
-    <xacro:wheel name = "front_right" path ="package://mobile_robot/meshes/left_tire.stl" x = "0.187" y = "-0.245"/>
-    <xacro:wheel name = "rear_left" path ="package://mobile_robot/meshes/right_tire.stl" x = "-0.187" y = "0.245"/>
-    <xacro:wheel name = "rear_right" path ="package://mobile_robot/meshes/left_tire.stl" x = "-0.187" y = "-0.245"/>
+    <!-- <xacro:wheel name = "front_left" path ="package://mobile_robot/meshes/right_tire.stl" x = "0.2" y = "0.25"/>
+    <xacro:wheel name = "front_right" path ="package://mobile_robot/meshes/left_tire.stl" x = "0.2" y = "-0.25"/>
+    <xacro:wheel name = "rear_left" path ="package://mobile_robot/meshes/right_tire.stl" x = "-0.2" y = "0.25"/>
+    <xacro:wheel name = "rear_right" path ="package://mobile_robot/meshes/left_tire.stl" x = "-0.2" y = "-0.25"/> -->
+    <xacro:wheel name = "front_left"    x = "0.2"     y = "0.25"/>
+    <xacro:wheel name = "front_right"   x = "0.2"     y = "-0.25"/>
+    <xacro:wheel name = "rear_left"     x = "-0.2"    y = "0.25"/>
+    <xacro:wheel name = "rear_right"    x = "-0.2"    y = "-0.25"/>
 </robot>
