Commit message: added the bot from fusion-360

File: description/gazebo_control.xacro (robot description, xacro)
@@ -1,10 +1,10 @@
 <?xml version="1.0"?>
 <robot xmlns:xacro="http://www.ros.org/wiki/xacro" name = "my_rover">
-    <gazebo>
+<!--    <gazebo>
         <plugin filename = "libgazebo_ros_diff_drive.so" name = "differential_drive_controller">
             <commandTopic>cmd_vel</commandTopic>
-            <odometryTopic>odom</odometryTopic>
+            <odometryTopic>odom</odometryTopic> -->
             <!-- <num_wheel_pairs> 2 </num_wheel_pairs> -->
-            <odometryFrame>odom</odometryFrame>
+            <!-- <odometryFrame>odom</odometryFrame>
             <odometrySource>world</odometrySource>
             <publishOdomTF>true</publishOdomTF>
@@ -16,8 +16,8 @@
             <updateRate>30</updateRate>
             <leftJoint>front_left_wheel_joint</leftJoint>
-            <rightJoint>front_right_wheel_joint</rightJoint>
+            <rightJoint>front_right_wheel_joint</rightJoint> -->
             <!-- <leftJoint>rear_left_wheel_joint</leftJoint> -->
             <!-- <rightJoint>rear_right_wheel_joint</rightJoint> -->
-            <wheelSeparation>0.5</wheelSeparation>
+            <!-- <wheelSeparation>0.5</wheelSeparation>
             <wheelDiameter>0.3</wheelDiameter>
             <wheelAcceleration>1</wheelAcceleration>
@@ -25,6 +25,6 @@
             <rosDebugLevel>na</rosDebugLevel>
         </plugin>
-    </gazebo>
-    <!-- <gazebo>
+    </gazebo> -->
+    <gazebo>
         <plugin name="skid_steer_drive_controller" filename="libgazebo_ros_skid_steer_drive.so">
             <updateRate>50.0</updateRate>
@@ -37,5 +37,5 @@
             <wheelDiameter>0.066</wheelDiameter>
             <robotBaseFrame>base_link</robotBaseFrame>
-            <torque>20</torque>
+            <torque>200</torque>
             <commandTopic>cmd_vel</commandTopic>
             <odometryTopic>odom</odometryTopic>
@@ -44,6 +44,6 @@
             <covariance_y>0.000100</covariance_y>
             <covariance_yaw>0.010000</covariance_yaw>
-            <broadcastTF>false</broadcastTF>
+            <broadcastTF>true</broadcastTF>
         </plugin>
-    </gazebo> -->
+    </gazebo>
 </robot>

File: urdf/rover.urdf.xacro (robot description, xacro)
@@ -15,5 +15,5 @@
     </xacro:macro> -->
     <!-- Dummy_link -->
-    <link name="base_footprint">
+    <!-- <link name="base_footprint">
     </link>
     <joint name="base_footprint_joint" type="fixed">
@@ -21,5 +21,5 @@
         <child link="base_footprint"/>
         <origin xyz="0.0 0.0 0.0" rpy="0.0 0.0 0.0"/>
-    </joint>
+    </joint> -->
     <!-- rover base link -->
     <link name="base_link">
@@ -154,13 +154,15 @@
         <!-- <origin xyz="${x} ${y} 0.15" rpy="0.0 0.0 0.0"/> -->
         <!-- <axis xyz="0.0 1.0 0.0"/> -->
-        <!-- <limit effort="100.0" lower="-3.14159" upper="3.14159" velocity="6.0"/>  -->
+        <limit effort="10000" velocity="1000"/>
     </joint>
     <!-- This block provides the simulator (Gazebo) with information on a few additional
     physical properties. See http://gazebosim.org/tutorials/?tut=ros_urdf for more-->
     <gazebo reference="${name}_wheel">
-      <mu1 value="200.0"/>
-      <mu2 value="100.0"/>
-      <kp value="500000.0" />
-      <kd value="1.0" />
+      <mu1 value="1"/>
+      <mu2 value="1"/>
+      <kp value="1000000.0" />
+      <kd value="100.0" />
+      <slip1 value="0.5" />
+      <slip2 value="0.5" />
       <material>Gazebo/Red</material>
     </gazebo>
